File: keyboard 3.kicad_pcb (KiCad board)
At the start: 2 copper layers, 9 parts, among them SW1 SW_Push, SW2 SW_Push, SW3 SW_Push, SW4 SW_Push, SW5 SW_Push, SW6 SW_Push, U1 XIAO-RP2040-DIP

Commit message: Add files via upload
Parts:
- added D10: 1N4148, Diode_THT:D_DO-35_SOD27_P7.62mm_Horizontal, F.Cu at (116.8, 63.5)
- added D11: 1N4148, Diode_THT:D_DO-35_SOD27_P7.62mm_Horizontal, F.Cu at (117.8, 83.8)
- added D12: 1N4148, Diode_THT:D_DO-35_SOD27_P7.62mm_Horizontal, F.Cu at (117.5, 103.2)
- added D13: 1N4148, Diode_THT:D_DO-35_SOD27_P7.62mm_Horizontal, F.Cu at (116.5, 122.0)
- added D14: 1N4148, Diode_THT:D_DO-35_SOD27_P7.62mm_Horizontal, F.Cu at (137.7, 63.5)
- added D15: 1N4148, Diode_THT:D_DO-35_SOD27_P7.62mm_Horizontal, F.Cu at (136.4, 82.5)
- added D16: 1N4148, Diode_THT:D_DO-35_SOD27_P7.62mm_Horizontal, F.Cu at (137.8, 102.5)
- added D17: 1N4148, Diode_THT:D_DO-35_SOD27_P7.62mm_Horizontal, F.Cu at (137.8, 122.2)
- added D18: SK6812, LED_SMD:LED_SK6812_PLCC4_5.0x5.0mm_P3.2mm, F.Cu at (65.0, 122.2)
- added D20: 1N4148, Diode_THT:D_DO-35_SOD27_P7.62mm_Horizontal, F.Cu at (55.5, 89.6)
- added D3: 1N4148, Diode_THT:D_DO-35_SOD27_P7.62mm_Horizontal, F.Cu at (82.5, 83.2)
- added D4: 1N4148, Diode_THT:D_DO-35_SOD27_P7.62mm_Horizontal, F.Cu at (80.9, 101.8)
- added D5: 1N4148, Diode_THT:D_DO-35_SOD27_P7.62mm_Horizontal, F.Cu at (77.9, 121.2)
- added D6: 1N4148, Diode_THT:D_DO-35_SOD27_P7.62mm_Horizontal, F.Cu at (100.4, 63.0)
- added D7: 1N4148, Diode_THT:D_DO-35_SOD27_P7.62mm_Horizontal, F.Cu at (98.7, 84.5)
- added D8: 1N4148, Diode_THT:D_DO-35_SOD27_P7.62mm_Horizontal, F.Cu at (98.2, 101.5)
- added D9: 1N4148, Diode_THT:D_DO-35_SOD27_P7.62mm_Horizontal, F.Cu at (98.4, 120.8)
- added SW10: SW_Push, Button_Switch_Keyboard:SW_Cherry_MX_1.00u_PCB, F.Cu at (124.0, 87.9)
- added SW11: SW_Push, Button_Switch_Keyboard:SW_Cherry_MX_1.00u_PCB, F.Cu at (124.0, 106.7)
- added SW12: SW_Push, Button_Switch_Keyboard:SW_Cherry_MX_1.00u_PCB, F.Cu at (124.2, 125.9)
- added SW13: SW_Push, Button_Switch_Keyboard:SW_Cherry_MX_1.00u_PCB, F.Cu at (143.2, 68.7)
- added SW14: SW_Push, Button_Switch_Keyboard:SW_Cherry_MX_1.00u_PCB, F.Cu at (143.2, 87.9)
- added SW15: SW_Push, Button_Switch_Keyboard:SW_Cherry_MX_1.00u_PCB, F.Cu at (143.2, 106.7)
- added SW16: SW_Push, Button_Switch_Keyboard:SW_Cherry_MX_1.00u_PCB, F.Cu at (143.5, 125.9)
- added SW17: RotaryEncoder, Rotary_Encoder:RotaryEncoder_Alps_EC11E-Switch_Vertical_H20mm, F.Cu at (55.2, 70.5)
- added SW7: SW_Push, Button_Switch_Keyboard:SW_Cherry_MX_1.00u_PCB, F.Cu at (104.8, 106.7)
- added SW8: SW_Push, Button_Switch_Keyboard:SW_Cherry_MX_1.00u_PCB, F.Cu at (105.0, 125.9)
- added SW9: SW_Push, Button_Switch_Keyboard:SW_Cherry_MX_1.00u_PCB, F.Cu at (124.0, 68.7)
- D1: value SK6812 -> 1N4148; footprint LED_SMD:LED_SK6812MINI_PLCC4_3.5x3.5mm_P1.75mm -> Diode_THT:D_DO-35_SOD27_P7.62mm_Horizontal
- D2: footprint LED_SMD:LED_SK6812MINI_PLCC4_3.5x3.5mm_P1.75mm -> LED_SMD:LED_SK6812_PLCC4_5.0x5.0mm_P3.2mm
- moved D2 114.4 mm to (65.0, 84.9)
- moved U1 102.9 mm to (62.0, 101.6), turned to 90 degrees
- moved SW4 79.0 mm to (85.8, 125.9)
- moved SW3 78.9 mm to (85.9, 106.8)
- moved SW5 68.3 mm to (105.0, 68.7)
- moved SW6 68.2 mm to (105.0, 87.7)
- moved D1 50.9 mm to (82.3, 61.8)
- moved SW1 49.3 mm to (86.0, 68.7)
- moved SW2 49.3 mm to (86.0, 87.7)
Connections:
- D1 pad 1: GND -> Net-(D1-K)
- D1 pad 2: Net-(D1-DIN) -> Net-(D1-A)
- D2 pad 2: Net-(D1-DOUT) -> Net-(D2-DIN)
- D2 pad 4: unconnected-(D2-DOUT-Pad4) -> Net-(D18-DIN)
- SW1 pad 1: GND -> Net-(U1-GPIO3/MOSI)
- SW1 pad 2: Net-(U1-GPIO7/SCL) -> Net-(D1-A)
- SW2 pad 1: GND -> Net-(U1-GPIO2/SCK)
- SW2 pad 2: Net-(U1-GPIO0/TX) -> Net-(D3-A)
- SW3 pad 1: GND -> Net-(U1-GPIO1/RX)
- SW3 pad 2: Net-(U1-GPIO1/RX) -> Net-(D4-A)
- SW4 pad 1: GND -> Net-(U1-GPIO4/MISO)
- SW4 pad 2: Net-(U1-GPIO2/SCK) -> Net-(D5-A)
- SW5 pad 1: GND -> Net-(U1-GPIO3/MOSI)
- SW5 pad 2: Net-(U1-GPIO4/MISO) -> Net-(D6-A)
- SW6 pad 1: GND -> Net-(U1-GPIO2/SCK)
- SW6 pad 2: Net-(U1-GPIO3/MOSI) -> Net-(D7-A)
- U1 pad 1: unconnected-(U1-GPIO26/ADC0/A0-Pad1) -> Net-(D20-K)
- U1 pad 13: unconnected-(U1-GND-Pad13) -> GND
- U1 pad 2: unconnected-(U1-GPIO27/ADC1/A1-Pad2) -> Net-(U1-GPIO27/ADC1/A1)
- U1 pad 3: unconnected-(U1-GPIO28/ADC2/A2-Pad3) -> Net-(D2-DIN)
- U1 pad 4: unconnected-(U1-GPIO29/ADC3/A3-Pad4) -> Net-(D1-K)
- U1 pad 5: Net-(D1-DIN) -> Net-(D6-K)
- U1 pad 6: Net-(U1-GPIO7/SCL) -> Net-(D10-K)
- U1 pad 7: Net-(U1-GPIO0/TX) -> Net-(D14-K)
Routing:
- net Net-(D14-K): track 0.00 -> 155.5 mm, vias 0 -> 2
- net Net-(D10-K): track 0.00 -> 120.1 mm, vias 0 -> 2
- net Net-(D6-K): track 0.00 -> 102.1 mm, vias 0 -> 1
- net Net-(U1-GPIO3/MOSI): track 0.00 -> 99.0 mm, vias 0 -> 1
- net Net-(U1-GPIO4/MISO): track 0.00 -> 98.4 mm
- net Net-(D1-K): track 0.00 -> 85.1 mm
- net Net-(U1-GPIO1/RX): track 0.00 -> 80.6 mm, vias 0 -> 3
- net Net-(U1-GPIO2/SCK): track 0.00 -> 80.3 mm, vias 0 -> 1
- net GND: track 0.00 -> 61.0 mm, vias 0 -> 1
- net +5V: track 0.00 -> 52.3 mm, vias 0 -> 3
- net Net-(D18-DIN): track 0.00 -> 44.8 mm, vias 0 -> 2
- net Net-(U1-GPIO27/ADC1/A1): track 0.00 -> 40.6 mm
- net Net-(D2-DIN): track 0.00 -> 24.1 mm
- net Net-(D20-K): track 0.00 -> 21.9 mm
- net Net-(D14-A): track 0.00 -> 14.6 mm
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Other:
- board outline added: 100 x 84 mm
- board text added: "bucket's hackpad"
